Commit message: add a robot model named whill_modelc

File: src/simulation/rtw_gazebo/xacro/roomba/base/base.xacro (robot description, xacro)
@@ -76,11 +76,4 @@
       <material name="purple"/>
     </visual>
-    <collision>
-      <geometry>
-        <mesh filename="package://rtw_gazebo/stl/Roomba_model.stl" />
-      </geometry>
-      <origin xyz="0 0 0" rpy="0 0 0"/>
-      <material name="purple"/>
-    </collision>
   </link>
   <gazebo reference="body_link">
