Commit message: modified coefficient of viscosity parameters of robot models

File: src/simulation/rtw_gazebo/xacro/dtw_robot/base/base.xacro (robot description, xacro)
@@ -13,4 +13,5 @@
       <child  link="${prefix}_link"/>
       <axis xyz="0 0 1" />
+      <dynamics damping="0.01"/>
     </joint>
     <transmission name="${prefix}_trans" type="SimpleTransmission">

File: src/simulation/rtw_gazebo/xacro/roomba/base/base.xacro (robot description, xacro)
@@ -16,6 +16,5 @@
       <child  link="${prefix}_link"/>
       <axis xyz="0 0 1" />
-      <limit velocity="12.0" effort="0.4" />
-      <dynamics damping="0.1"/>
+      <dynamics damping="0.01"/>
     </joint>
     <transmission name="${prefix}_trans">
